File: mcu.kicad_sch (KiCad schematic)
At the start: 45 parts, among them SW1 SW_Push, SW2 Volume Up, SW3 Volume Down, SW4 Play/Pause, SW5 Power Switch, U6 CH340X, U7 ESP32-WROOM-32, U8 MAX98357A

Commit message: Remove Boost
Connections:
- net VREG_5V is gone; now on net VREG_3.3V: C16.2, C17.2, U8.7 (VDD), U8.8 (VDD)
Changed lines of the file:
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@@
+		)
+	)
+	(global_label "VREG_3.3V"
+		(shape input)
+		(at 204.47 110.49 0)
+		(fields_autoplaced yes)
+		(effects
+			(font
+				(size 1.27 1.27)
+			)
+			(justify left)
+		)
+		(property "Intersheetrefs" "${INTERSHEET_REFS}"
+			(at 217.3128 110.49 0)
+			(effects
+				(font
+					(size 1.27 1.27)
+				)
+				(justify left)
+				(hide yes)
+			)
 		)
 	)
@@
 			(effects
 				(font
-					(size 1.27 1.27)
-				)
-				(justify left)
-				(hide yes)
-			)
-		)
-	)
-	(global_label "VREG_5V"
-		(shape input)
-		(at 204.47 110.49 0)
-		(fields_autoplaced yes)
-		(effects
-			(font
-				(size 1.27 1.27)
-			)
-			(justify left)
-		)
-		(property "Intersheetrefs" "${INTERSHEET_REFS}"
-			(at 215.4985 110.49 0)
-			(effects
-				(font

Commit message: Update the MCU sheet
Parts:
- removed C14: 0.1uF, Capacitor_SMD:C_0603_1608Metric_Pad1.08x0.95mm_HandSolder, symbol Device:C
- removed C23: 100pF, Capacitor_SMD:C_0603_1608Metric_Pad1.08x0.95mm_HandSolder, symbol Device:C
- added C4: 0.1uF, Capacitor_SMD:C_0603_1608Metric_Pad1.08x0.95mm_HandSolder, symbol Device:C
- renumbered C11 to C1, C12 to C2, C13 to C3, C16 to C5, C17 to C6, C15 to C7, D3 to D1, D4 to D2, D5 to D3, D6 to D4, D7 to D5, R14 to R1, R19 to R10, R32 to R11, R20 to R12, R21 to R13, R22 to R14, R23 to R15, R24 to R16, R15 to R2, R30 to R3, R16 to R4, R31 to R5, R17 to R6, R25 to R7, R18 to R8, R26 to R9, TP12 to TP1, TP13 to TP2, TP2 to TP3, TP1 to TP4, TP14 to TP5, TP15 to TP6, TP16 to TP7, U6 to U1, U7 to U2, U8 to U3
Connections:
- net GND: now also C4.1
- net VREG_3.3V: now also C4.2
- net AMP_SDM: now reaches U2.9 (IO33)
- net AMP_SDM: now also U3.4 (~{SD_MODE})
- net at R11.1, U1.7 (VCC): now also U1.10 (V3)
- no-connect marks 16 -> 14
Other:
- note removed: "TODO check filter caps"
- moved on the sheet: C5, C6, C7, LS1, R13, R14, R15, R16, SW5, TP5, TP6, TP7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

Commit message: Update the USB-C symbol to match the actual part
Parts:
- added H3, H4, H5, H6: MountingHole, MountingHole:MountingHole_2.2mm_M2_Pad_Via, symbol Mechanical:MountingHole
- R22: renamed from R14; footprint (none) -> Resistor_SMD:R_0603_1608Metric_Pad0.98x0.95mm_HandSolder
- R23: renamed from R15; footprint (none) -> Resistor_SMD:R_0603_1608Metric_Pad0.98x0.95mm_HandSolder
- R24: renamed from R16; footprint (none) -> Resistor_SMD:R_0603_1608Metric_Pad0.98x0.95mm_HandSolder
- R25: renamed from R7; footprint (none) -> Resistor_SMD:R_0603_1608Metric_Pad0.98x0.95mm_HandSolder
- R26: renamed from R9; footprint (none) -> Resistor_SMD:R_0603_1608Metric_Pad0.98x0.95mm_HandSolder
- R30: renamed from R3; footprint (none) -> Resistor_SMD:R_0603_1608Metric_Pad0.98x0.95mm_HandSolder
- R31: renamed from R5; footprint (none) -> Resistor_SMD:R_0603_1608Metric_Pad0.98x0.95mm_HandSolder
- R32: renamed from R11; footprint (none) -> Resistor_SMD:R_0603_1608Metric_Pad0.98x0.95mm_HandSolder
- TP1: renamed from TP4; footprint (none) -> TestPoint:TestPoint_Pad_D2.5mm
- TP12: renamed from TP1; footprint (none) -> TestPoint:TestPoint_Pad_D2.5mm
- TP13: renamed from TP2; footprint (none) -> TestPoint:TestPoint_Pad_D2.5mm
- TP14: renamed from TP5; footprint (none) -> TestPoint:TestPoint_Pad_D2.5mm
- TP15: renamed from TP6; footprint (none) -> TestPoint:TestPoint_Pad_D2.5mm
- TP16: renamed from TP7; footprint (none) -> TestPoint:TestPoint_Pad_D2.5mm
- TP2: renamed from TP3; footprint (none) -> TestPoint:TestPoint_Pad_D2.5mm
- renumbered C1 to C11, C2 to C12, C3 to C13, C7 to C15, C5 to C16, C6 to C17, C4 to C7, D1 to D3, D2 to D4, D3 to D5, D4 to D6, D5 to D7, R1 to R14, R2 to R15, R4 to R16, R6 to R17, R8 to R18, R10 to R19, R12 to R20, R13 to R21, U1 to U6, U2 to U7, U3 to U8

Commit message: Put component families together on PCB
Parts:
- added C8: 1nF, Capacitor_SMD:C_0603_1608Metric_Pad1.08x0.95mm_HandSolder, symbol Device:C
- TP1, TP12, TP13, TP14, TP15, TP16, TP2: footprint TestPoint:TestPoint_Pad_D2.5mm -> TestPoint:TestPoint_Pad_D1.5mm
Connections:
- net GND: now also C8.1
- net VREG_3.3V: now also C8.2
Other:
- moved on the sheet: C16, C17

Commit message: Update LDO and make some visual tweaks suggested by conor
Connections:
- net Enable: now reaches C11.2, C13.1, R14.2, SW1.2, U7.3 (EN)
Other:
- note added: "EN Circuit 1ms Time Constant"
- note added: "Speaker Driver + Speaker"
- note added: "Speaker Power 3W"
- moved on the sheet: C11, C12, C13, C16, C17, C8, LS1, R14, R22, R23, R24, SW1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

Commit message: Mostly finished schematic and pcb, getting codex to review it now
Parts:
- renumbered C7 to C14, C16 to C15, C17 to C16, C15 to C17, C8 to C18, H3 to H1, H4 to H2, H5 to H3, H6 to H4, R14 to R16, R15 to R17, R30 to R18, R16 to R19, R31 to R20, R17 to R21, R25 to R22, R18 to R23, R26 to R24, R19 to R25, R32 to R26, R20 to R27, R21 to R28, R22 to R29, R23 to R30, R24 to R31, TP13 to TP10, TP2 to TP11, TP1 to TP12, TP14 to TP13, TP15 to TP14, TP16 to TP15, TP12 to TP9, U6 to U5, U7 to U6, U8 to U7
Connections:
- net Speaker-: now reaches LS1.2, U7.10 (OUT-)
- net Speaker+: now reaches LS1.1, U7.9 (OUT+)
