File: power.kicad_sch (KiCad schematic)
At the start: 43 parts, among them J2 UJ20-C-H-G-SMT-1-P16-TR, U1 LT1963AxST-3.3, U2 MCP73871, U4 MAX17048G_T10, U5 USBLC6-2SC6

Commit message: Mostly finished schematic and pcb, getting codex to review it now
Parts:
- renumbered C6 to C1, C1 to C10, C5 to C2, C4 to C3, C19 to C4, C22 to C5, C21 to C6, C18 to C7, C3 to C8, C2 to C9, J2 to J1, R5 to R10, R6 to R11, R7 to R12, R8 to R13, R3 to R14, R33 to R15, R27 to R2, R2 to R3, R28 to R4, R29 to R5, R4 to R6, R9 to R7, R10 to R8, R11 to R9, TP4 to TP1, TP8 to TP2, TP9 to TP3, TP7 to TP4, TP3 to TP5, TP10 to TP6, TP5 to TP7, TP6 to TP8, TP_VSYS_LDO to TP_VSYS_LDO1, U4 to U1, U1 to U3, U5 to U4
Connections:
- net USBtoSchottky+: now reaches J1.A6 (D_P), J1.B6 (D2_P), U4.3 (I/O2)
- net USBtoSchottky-: now reaches J1.A7 (D_N), J1.B7 (D2_N), U4.1 (I/O1)
